File: pcb-n-as5600.kicad_sch (KiCad schematic)
At the start: 26 parts, among them J1 Conn_01x04, J2 Conn_01x04_Pin, J5 Conn_01x04, J6 USB_C_Receptacle_USB2.0_14P, SW2 SW_Push, SW3 SW_Push, U4 AS5600, U5 STM32F103C8Tx, U6 AP2112K-3.3, Y2 8MHz

Commit message: changes to PCB, schematic
changed netlist, changed regulator used, changed PCB
Parts:
- removed C15, C9: 100nF, Capacitor_SMD:C_0603_1608Metric_Pad1.08x0.95mm_HandSolder, symbol Device:C
- removed J1: Conn_01x04, Connector_PinHeader_1.27mm:PinHeader_1x04_P1.27mm_Vertical, symbol Connector_Generic:Conn_01x04
- removed J5: Conn_01x04, Connector_PinSocket_2.00mm:PinSocket_1x04_P2.00mm_Vertical, symbol Connector_Generic:Conn_01x04
- removed SW2, SW3: SW_Push, Button_Switch_SMD:SW_SPST_B3U-1000P, symbol Switch:SW_Push
- removed U6: AP2112K-3.3, Package_TO_SOT_SMD:SOT-23-5, symbol Regulator_Linear:AP2112K-3.3
- added C1, C2, C3, C4: 100nF, Capacitor_SMD:C_0603_1608Metric_Pad1.08x0.95mm_HandSolder, symbol Device:C
- added J1, J3: Conn_01x04_Pin, Connector_PinSocket_2.00mm:PinSocket_1x04_P2.00mm_Vertical, symbol Connector:Conn_01x04_Pin
- added R2: 5k1, Resistor_SMD:R_0603_1608Metric_Pad0.98x0.95mm_HandSolder, symbol Device:R
- added R3, R4: 10k, Resistor_SMD:R_0603_1608Metric_Pad0.98x0.95mm_HandSolder, symbol Device:R
- added S1, S2: TS09-63-25-WT-160-SMT-TR, TS09-63-25-WT-160-SMT-TR:SW_TS09-63-25-WT-160-SMT-TR, symbol TS09 Switch:TS09-63-25-WT-160-SMT-TR
- added U1: AMS1117, Package_TO_SOT_SMD:SOT-223-3_TabPin2, symbol Regulator_Linear:AMS1117
- J6: footprint Connector_USB:USB_C_Receptacle_HRO_TYPE-C-31-M-12 -> Connector_USB:USB_C_Receptacle_GCT_USB4105-xx-A_16P_TopMnt_Horizontal
Connections:
- net 3.3V: now also J1.3 (Pin_3), J3.3 (Pin_3), R2.1; no longer C10.1, C11.1, C13.1, C14.1, C7.1, C7.2, C8.1, J6.A1 (GND), J6.A12 (GND), J6.B1 (GND), J6.B12 (GND), R1.2, R11.1, R8.1, R9.2, U4.1 (VDD5V), U4.2 (VDD3V3), U4.4 (GND), U5.23 (VSS), U5.35 (VSS), U5.47 (VSS)
- net BOOTO: now also S1.1
- net MCU_D+: now also R2.2
- net NRST: now also S2.1
- net RX: now also J3.2 (Pin_2)
- net SCLK: now also J1.2 (Pin_2)
- net SWDIO: now also J1.1 (Pin_1)
- net TX: now also J3.1 (Pin_1)
- net +3.3V: now reaches U5.1 (VBAT)
- net +3.3V: now also C11.1, C7.1, R9.2, U4.1 (VDD5V), U4.2 (VDD3V3), U5.24 (VDD), U5.36 (VDD), U5.48 (VDD), C1.1, C2.1, C3.1, R4.1, U1.2 (VO)
- net GND: now reaches U5.8 (VSSA)
- net GND: now also C10.1, C11.2, C13.1, C14.1, C7.2, C8.1, J6.A1 (GND), J6.A12 (GND), J6.B1 (GND), J6.B12 (GND), R1.2, R11.1, R8.1, U4.4 (GND), U5.23 (VSS), U5.35 (VSS), U5.47 (VSS), C1.2, C2.2, C3.2, C4.2, J1.4 (Pin_4), J3.4 (Pin_4), R3.2, S1.2, S2.2
- removed net VDD: C11.2, U5.24 (VDD), U5.36 (VDD), U5.48 (VDD)
- new net: R3.1, R4.2, U1.1 (ADJ)
- new net +5V: C4.1, U1.3 (VI)
- no-connect marks 26 -> 24
Other:
- note added: "AMS1117"
- note removed: "AP2112K-3.3"
- moved on the sheet: C11, R13, R9

Commit message: addition of mount holes
rechecked voltage connections as well, and added
Parts:
- added H1, H2, H3, H4: MountingHole, MountingHole:MountingHole_3.2mm_M3_Pad, symbol Mechanical:MountingHole
Connections:
- net 3.3V is gone; now on net +3.3V: J1.3 (Pin_3), J3.3 (Pin_3), R13.1, R16.2, R2.1, R7.1

Commit message: final pcb with proper connections
removed UART due to lack of use, connections are correct, slight silk screen issue, final draft
Parts:
- removed J3: Conn_01x04_Pin, Connector_PinSocket_2.00mm:PinSocket_1x04_P2.00mm_Vertical, symbol Connector:Conn_01x04_Pin
Connections:
- net RX: no longer names the net of U5.31 (PA10)
- net TX: no longer names the net of U5.30 (PA9)
- no-connect marks 24 -> 26
Other:
- note removed: "UART"
