File: pcb-n-as5600.kicad_pcb (KiCad board)
At the start: 2 copper layers, 46.5 x 46.9 mm, 34 parts, among them J1 Conn_01x04_Pin, J2 Conn_01x04_Pin, J6 USB_C_Receptacle_USB2.0_14P, U1 AMS1117, U4 AS5600, U5 STM32F103C8Tx, Y2 8MHz

Commit message: final final
Parts:
- moved H4 0.71 mm to (170.8, 104.8)
- moved H3 0.61 mm to (170.6, 68.3)
- moved H1 0.60 mm to (133.9, 105.3)
Other:
- board size 46.5 x 46.9 mm -> 46.5 x 46.6 mm
